File: Design/bldc/CAN.kicad_sch (KiCad schematic)
At the start: 0 parts

Commit message: Adding components to schematic
Parts:
- added C? (x2): 2.2u, symbol Device:C_Small
- added JP?: Jumper, symbol Jumper:Jumper_2_Bridged
- added R?: 120, symbol Device:R
- added U?: TJA1051TK-3, Package_DFN_QFN:DFN-8-1EP_3x3mm_P0.65mm_EP1.55x2.4mm, symbol Interface_CAN_LIN:TJA1051TK-3
Connections:
- new net: JP?.1 (A), R?.1
- new net +3.3V: C?.1, U?.5 (VIO)
- new net +5V: C?.1, U?.3 (VCC)
- new net CANH: JP?.2 (B), U?.7 (CANH)
- new net CANL: R?.2, U?.6 (CANL)
- new net CANRX: U?.4 (RXD)
- new net CANTX: U?.1 (TXD)
- new net GND: C?.2, C?.2, U?.2 (GND), U?.8 (S), U?.9 (GND)
Other:
- note added: "Optional 120Ω"
