File: Design/bldc/STM32F4.kicad_sch (KiCad schematic)
At the start: 0 parts

Commit message: Adding components to schematic
Other:
- title: (none) -> BLDC motor controller
Changed lines of the file:
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@@
 (kicad_sch (version 20211123) (generator eeschema)
   (paper "A4")
+  (title_block
+    (title "BLDC motor controller")
+    (date "2022-12-11")
+    (rev "1.0.0")
+  )
+  (hierarchical_label "VBatt" (shape input) (at 70.485 37.465 180)
+    (effects (font (size 1.27 1.27)) (justify right))
+  )
 )
