File: Design/bldc/gate_drivers.kicad_sch (KiCad schematic)
At the start: 0 parts

Commit message: Adding components to schematic
Other:
- title: (none) -> BLDC motor controller
Changed lines of the file:
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@@
 (kicad_sch (version 20211123) (generator eeschema)
   (paper "A4")
+  (title_block
+    (title "BLDC motor controller")
+    (date "2022-12-11")
+    (rev "1.0.0")
+  )
 )
