File: Design/bldc/hall_filters.kicad_sch (KiCad schematic)
At the start: 0 parts

Commit message: Adding components to schematic
Parts:
- added C? (x3): 4.7nF, symbol Device:C
- added C?: 100nF, symbol Device:C
- added R? (x3): 2.2k, symbol Device:R
- added R? (x4): 10k, symbol Device:R
Connections:
- new net +3.3V: R?.1, R?.1, R?.1, R?.1
- new net GND: C?.2, C?.2, C?.2, C?.2
- new net HALL1_IN: R?.1, R?.2
- new net HALL1_OUT: C?.1, R?.2
- new net HALL2_IN: R?.1, R?.2
- new net HALL2_OUT: C?.1, R?.2
- new net HALL3_IN: R?.1, R?.2
- new net HALL3_OUT: C?.1, R?.2
- new net TEMP_IN: C?.1, R?.2
Other:
- title: (none) -> BLDC motor controller
