File: Design/gate_drivers.kicad_sch (KiCad schematic)
At the start: 0 parts

Commit message: schematic updates
Parts:
- added U? (x3): UCC2721xA, symbol infineon:UCC2720xA
Connections:
- new net: U?.7 (VSS), U?.9 (PowerPad) (x3)
Changed lines of the file:
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@@
     (rev "1.0.0")
   )
+  (symbol (lib_id "infineon:UCC2720xA") (at 132.715 46.355 0) (unit 1)
+    (in_bom yes) (on_board yes) (fields_autoplaced)
+    (property "Reference" "U?" (id 0) (at 135.255 36.83 0)
+      (effects (font (size 1.524 1.524)))
+    )
+    (property "Value" "UCC2721xA" (id 1) (at 135.255 40.64 0)
+      (effects (font (size 1.524 1.524)))
+    )
+    (property "Footprint" "" (id 2) (at 132.715 46.355 0)
+      (effects (font (size 1.524 1.524)) hide)
+    )
+    (property "Datasheet" "" (id 3) (at 132.715 46.355 0)
+      (effects (font (size 1.524 1.524)) hide)
+    )
+    (pin "1")
+    (pin "2")
+    (pin "3")
+    (pin "4")
+    (pin "5")
+    (pin "6")
+    (pin "7")
+    (pin "8")
+    (pin "9")
+  )
+  (symbol (lib_id "infineon:UCC2720xA") (at 133.985 102.235 0) (unit 1)
+    (in_bom yes) (on_board yes) (fields_autoplaced)
+    (property "Reference" "U?" (id 0) (at 136.525 92.71 0)
+      (effects (font (size 1.524 1.524)))
+    )
+    (property "Value" "UCC2721xA" (id 1) (at 136.525 96.52 0)
+      (effects (font (size 1.524 1.524)))
+    )
+    (property "Footprint" "" (id 2) (at 133.985 102.235 0)
+      (effects (font (size 1.524 1.524)) hide)
+    )
+    (property "Datasheet" "" (id 3) (at 133.985 102.235 0)
+      (effects (font (size 1.524 1.524)) hide)
+    )
+    (pin "1")
+    (pin "2")
+    (pin "3")
+    (pin "4")
+    (pin "5")
+    (pin "6")
+    (pin "7")
+    (pin "8")
+    (pin "9")
+  )
+  (symbol (lib_id "infineon:UCC2720xA") (at 133.35 75.565 0) (unit 1)
+    (in_bom yes) (on_board yes) (fields_autoplaced)
+    (property "Reference" "U?" (id 0) (at 135.89 66.04 0)
+      (effects (font (size 1.524 1.524)))
+    )
+    (property "Value" "UCC2721xA" (id 1) (at 135.89 69.85 0)
+      (effects (font (size 1.524 1.524)))
+    )
+    (property "Footprint" "" (id 2) (at 133.35 75.565 0)
+      (effects (font (size 1.524 1.524)) hide)
+    )
+    (property "Datasheet" "" (id 3) (at 133.35 75.565 0)
+      (effects (font (size 1.524 1.524)) hide)
+    )
+    (pin "1")
+    (pin "2")
+    (pin "3")
+    (pin "4")
+    (pin "5")
+    (pin "6")
+    (pin "7")
+    (pin "8")
+    (pin "9")
+  )
 )
