File: Design/gate_drivers.kicad_sch (KiCad schematic)
At the start: 0 parts

Commit message: gate driver
Parts:
- added C? (x7): 100n, symbol Device:C_Small
- added C? (x3): 2.2u, symbol Device:C_Small
- added U?: DRV8328C, symbol TI:DRV8328C
Connections:
- new net: C?.1, C?.1, C?.1, C?.1, U?.3 (CPH)
- new net: C?.2, C?.2, C?.2, C?.2, U?.2 (CPL)
- new net: C?.2, U?.9 (BSTB)
- new net: C?.2, C?.2, U?.4 (GVDD)
- new net: C?.2, U?.13 (BSTC)
- new net: C?.2, U?.5 (BSTA)
- new net +3.3V: C?.1, U?.19 (AVDD)
- new net +BATT: U?.1 (PVDD)
- new net DRVOFF: U?.18 (DRVOFF)
- new net GH_A: U?.7 (GHA)
- new net GH_B: U?.11 (GHB)
- new net GH_C: U?.15 (GHC)
- new net GL_A: U?.8 (GLA)
- new net GL_B: U?.12 (GLB)
- new net GL_C: U?.16 (GLC)
- new net GND: C?.1, C?.1, C?.2, U?.28 (GND), U?.29 (GND)
- new net HS_A_TTL: U?.22 (INHA)
- new net HS_B_TTL: U?.21 (INHB)
- new net HS_C_TTL: U?.20 (INHC)
- new net LSS: U?.17 (LSS)
- new net LS_A_TTL: U?.25 (INLA)
- new net LS_B_TTL: U?.24 (INLB)
- new net LS_C_TTL: U?.23 (INLC)
- new net PHASE_A_SOURCE: C?.1, U?.6 (SHA)
- new net PHASE_B_SOURCE: C?.1, U?.10 (SHB)
- new net PHASE_C_SOURCE: C?.1, U?.14 (SHC)
- new net nFAULT: U?.27 (nFAULT)
- new net nSLEEP: U?.26 (nSLEEP)
Other:
- note added: "WOULD RATHER USE THE DRV8323RH GATE DRIVER. UNFORTUNATELY SUPPLY SHORTAGES ARE PREVENTING THAT."

Commit message: drv8323RH
Parts:
- removed C? (x7): 100n, symbol Device:C_Small
- removed C? (x3): 2.2u, symbol Device:C_Small
- removed U?: DRV8328C, symbol TI:DRV8328C
- added C? (x3): 4.7uF_100V, symbol Device:C
- added C? (x2): 100n, symbol Device:C_Small
- added C? (x2): 1u, symbol Device:C_Small
- added R?: 1M, symbol Device:R
- added R?: 10k, symbol Device:R
- added R? (x2): 39k, symbol Device:R
- added U?: DRV8323RH, Package_DFN_QFN:QFN-48-1EP_7x7mm_P0.5mm_EP5.15x5.15mm_ThermalVias, symbol TI:DRV8323RH
Connections:
- net +3.3V: now also C?.1, R?.1, U?.26 (VREF)
- net +BATT: now also C?.1, C?.2, C?.2, C?.2, U?.6 (VM), U?.7 (VDRAIN)
- net GH_A: now also U?.8 (GHA)
- net GH_B: now also U?.17 (GHB)
- net GH_C: now also U?.18 (GHC)
- net GL_A: now also U?.10 (GLA)
- net GL_B: now also U?.15 (GLB)
- net GL_C: now also U?.20 (GLC)
- net GND: now also C?.1, C?.1, C?.1, C?.2, R?.2, U?.12 (SNA), U?.13 (SNB), U?.2 (PGND), U?.22 (SNC), U?.27 (DGND), U?.49 (GND)
- net HS_A_TTL: now also U?.37 (INHA)
- net HS_B_TTL: now also U?.39 (INHB)
- net HS_C_TTL: now also U?.41 (INHC)
- net LS_A_TTL: now also U?.38 (INLA)
- net LS_B_TTL: now also U?.40 (INLB)
- net LS_C_TTL: now also U?.42 (INLC)
- net nFAULT: now also R?.2, U?.28 (nFAULT)
- new net: R?.1, U?.32 (GAIN)
- new net: R?.1, U?.31 (VDS)
- new net: R?.1, R?.2
- new net: C?.2, U?.5 (VCP)
- new net: C?.1, U?.3 (CPL)
- new net: C?.2, U?.4 (CPH)
- new net: C?.1, U?.35 (AGND)
- new net CAL: U?.34 (CAL)
- new net DVDD: C?.2, R?.2, U?.29 (MODE), U?.30 (IDRIVE), U?.36 (DVDD)
- new net ENABLE: U?.33 (ENABLE)
- new net PHASEA_FB: U?.25 (SOA)
- new net PHASEB_FB: U?.24 (SOB)
- new net PHASEC_FB: U?.23 (SOC)
- new net PHASE_A_OUT: U?.9 (SHA)
- new net PHASE_B_OUT: U?.16 (SHB)
- new net PHASE_C_OUT: U?.19 (SHC)
- new net SPA: U?.11 (SPA)
- new net SPB: U?.14 (SPB)
- new net SPC: U?.21 (SPC)
- no-connect marks 0 -> 1
Other:
- note added: "1.88V ACROSS VDRAIN AND SHx TRIPS OCP"
- note added: "20V/V AMPLIFIER GAIN"
- note added: "INDEPENDENT PWM MODE"
- note added: "MAX GATE SOURCE/SINK CURRENT"

Commit message: 3.3v reg
Parts:
- added C? (x2): 100n, symbol Device:C_Small
- added C?: 4.7uF_100V, symbol Device:C
- added D?: B160-E3, Diode_SMD:D_SMA, symbol Diode:B160-E3
- added L?: 27u, symbol Device:L_Small
- added R? (x3): 39k, symbol Device:R
- added R?: 33k, symbol Device:R_Small
- added R?: 10k, symbol Device:R_Small
Connections:
- net +3.3V: now also C?.2, L?.2, R?.1
- net +BATT: now also U?.47 (VIN), C?.2, R?.2
- net GND: now also C?.1, C?.1, D?.2 (A), R?.1
- net V_FB: now reaches U?.1 (FB)
- net V_FB: now also R?.2, R?.2
- net at U?.44 (CB): now also C?.1
- net at U?.45 (SW): now also C?.2, D?.1 (K), L?.1
- net at U?.48 (nSHD): now also R?.1
- new net: R?.1, R?.2 (x2)
Other:
- note added: "24uH L_{o min} 183mA ripple 0.69 I_{L-peak} 0.602 I_{L-RMS}"
- note added: "C_{bootstrap} = 200nF @ >=10V rating"
- note added: "C_{in} = 4.7uF @ 100V"
- note added: "C_{out} > 16.4µF per EQ. 5 C_{out} > 12.8µF per EQ. 6 C_{out} > 0.99uF per EQ. 7 R_{esr} < 0.180Ω per EQ. 8"
- note added: "schottkey diode: V_{breakdown} = 62.5 V I_{rate} = 0.5A to 1A"

Commit message: SWD debugger
Connections:
- net GND: now also U?.43 (BGND)
Changed lines of the file:
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@@
     (pin "2")
+  )
+  (symbol (lib_id "power:GND") (at 156.845 111.125 90) (unit 1)
+    (in_bom yes) (on_board yes) (fields_autoplaced)
+    (property "Reference" "#GND" (id 0) (at 163.195 111.125 0)
+      (effects (font (size 1.27 1.27)) hide)
+    )
+    (property "Value" "GND" (id 1) (at 161.29 111.125 0)
+      (effects (font (size 1.27 1.27)) hide)
+    )
+    (property "Footprint" "" (id 2) (at 156.845 111.125 0)
+      (effects (font (size 1.27 1.27)) hide)
+    )
+    (property "Datasheet" "" (id 3) (at 156.845 111.125 0)
+      (effects (font (size 1.27 1.27)) hide)
+    )
+    (pin "1")
   )
   (symbol (lib_id "Device:C_Small") (at 163.195 113.665 90) (unit 1)

Commit message: Updating schematic
Parts:
- gave numbers to parts that had none: 22
Other:
- note removed: "WOULD RATHER USE THE DRV8323RH GATE DRIVER. UNFORTUNATELY SUPPLY SHORTAGES ARE PREVENTING THAT."
