File: Design/CAN.kicad_sch (KiCad schematic)
At the start: 5 parts

Commit message: schematic updates
Other:
- moved on the sheet: C?, JP?, R?, U?

Commit message: MOSFETS
Parts:
- removed C?: 2.2u, symbol Device:C_Small
- removed U?: TJA1051TK-3, Package_DFN_QFN:DFN-8-1EP_3x3mm_P0.65mm_EP1.55x2.4mm, symbol Interface_CAN_LIN:TJA1051TK-3
- added U?: SN65HVD232, Package_SO:SOIC-8_3.9x4.9mm_P1.27mm, symbol Interface_CAN_LIN:SN65HVD232
Connections:
- net +3.3V: now also U?.3 (VCC)
- net CANH: now also U?.7 (CANH)
- net CANL: now also U?.6 (CANL)
- net CANRX: now also U?.4 (R)
- net CANTX: now also U?.1 (D)
- net GND: now also U?.2 (GND)
Other:
- moved on the sheet: C?

Commit message: Updating schematic
Parts:
- JP1: renamed from JP?; value Jumper -> 0.1" Jumper
- gave numbers to parts that had none: 3
Changed lines of the file:
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@@
   (symbol (lib_id "Device:C_Small") (at 118.745 86.995 0) (unit 1)
     (in_bom yes) (on_board yes)
-    (property "Reference" "C?" (id 0) (at 119.38 85.09 0)
+    (property "Reference" "C2" (id 0) (at 119.38 85.09 0)
       (effects (font (size 1.27 1.27)) (justify left))
     )
@@
   (symbol (lib_id "Device:R") (at 187.96 98.425 0) (unit 1)
     (in_bom yes) (on_board yes)
-    (property "Reference" "R?" (id 0) (at 189.23 97.79 0)
+    (property "Reference" "R3" (id 0) (at 189.23 97.79 0)
       (effects (font (size 1.27 1.27)) (justify left))
     )
@@
   (symbol (lib_id "Jumper:Jumper_2_Bridged") (at 187.96 86.995 90) (unit 1)
     (in_bom yes) (on_board yes)
-    (property "Reference" "JP?" (id 0) (at 189.23 86.995 90)
+    (property "Reference" "JP1" (id 0) (at 189.23 86.995 90)
       (effects (font (size 1.27 1.27)) (justify right))
     )
-    (property "Value" "Jumper" (id 1) (at 189.23 88.2649 90)
+    (property "Value" "0.1\" Jumper" (id 1) (at 189.23 88.2649 90)
       (effects (font (size 1.27 1.27)) (justify right) hide)
     )
@@
   (symbol (lib_id "power:GND") (at 151.765 105.41 0) (unit 1)
     (in_bom yes) (on_board yes) (fields_autoplaced)
-    (property "Reference" "#GND" (id 0) (at 151.765 111.76 0)
+    (property "Reference" "#GND08" (id 0) (at 151.765 111.76 0)
       (effects (font (size 1.27 1.27)) hide)
     )
@@
   (symbol (lib_id "power:+3.3V") (at 118.745 76.2 0) (unit 1)
     (in_bom yes) (on_board yes)
-    (property "Reference" "#PWR3.3" (id 0) (at 118.745 80.01 0)
+    (property "Reference" "#PWR05" (id 0) (at 118.745 80.01 0)
       (effects (font (size 1.27 1.27)) hide)
     )
@@
   (symbol (lib_id "Interface_CAN_LIN:SN65HVD232") (at 151.765 89.535 0) (unit 1)
     (in_bom yes) (on_board yes) (fields_autoplaced)
-    (property "Reference" "U?" (id 0) (at 153.7844 79.375 0)
+    (property "Reference" "U1" (id 0) (at 153.7844 79.375 0)
       (effects (font (size 1.27 1.27)) (justify left))
     )
