File: Design/bldc.kicad_sch (KiCad schematic)
At the start: 10 parts

Commit message: SWD debugger
Parts:
- added J?: SWD, symbol Connector_Generic:Conn_01x05
Connections:
- net +3.3V: now also J?.5 (Pin_5)
- net GND: now also J?.3 (Pin_3)
- net MCU/NRST: now also J?.1 (Pin_1)
- new net MCU/SWCLK: J?.4 (Pin_4)
- new net MCU/SWDIO: J?.2 (Pin_2)
Other:
- sheet MCU ports: added CAL, ENABLE, SWCLK, SWDIO, nFAULT; removed none

Commit message: Updating schematic
Parts:
- added J6: USART, symbol Connector_Generic:Conn_01x06
- J1, J2, J7, J8, J9: renamed from J?; now left out of the parts list
- gave numbers to parts that had none: 6
Connections:
- net +3.3V: now also J6.3 (Pin_3)
- net GND: now also J6.1 (Pin_1)
- new net MCU/USART_CTS: J6.2 (Pin_2)
- new net MCU/USART_RTS: J6.6 (Pin_6)
- new net MCU/USART_RX: J6.5 (Pin_5)
- new net MCU/USART_TX: J6.4 (Pin_4)
Other:
- sheet MCU ports: added USART_CTS, USART_RTS, USART_RX, USART_TX; removed none

Commit message: adding caps
Other:
- sheet MCU ports: added MOSFET_Temp; removed none
- sheet Power MOSFETS ports: added MOSFET_Temp; removed none
Changed lines of the file:
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@@
+    (stroke (width 0) (type default) (color 0 0 0 0))
+  )
+  (wire (pts (xy 133.35 115.57) (xy 191.77 115.57))
     (stroke (width 0) (type default) (color 0 0 0 0))
   )
@@
       (effects (font (size 1.27 1.27)) (justify left))
     )
+    (pin "MOSFET_Temp" output (at 191.77 115.57 180)
+      (effects (font (size 1.27 1.27)) (justify left))
+    )
   )
   (sheet (at 83.82 36.83) (size 49.53 125.73) (fields_autoplaced)
@@
     (pin "USART_CTS" input (at 83.82 149.86 180)
       (effects (font (size 1.27 1.27)) (justify left))
+    )
+    (pin "MOSFET_Temp" input (at 133.35 115.57 0)
+      (effects (font (size 1.27 1.27)) (justify right))
     )
   )
@@
       (reference "#GND031") (unit 1) (value "GND") (footprint "")
     )
+    (path "/07a796a7-971a-46f8-be0a-5ed59c09f1bb/7f1a27a0-ee12-465d-82a7-694ac3a112e7"
+      (reference "#GND032") (unit 1) (value "GND") (footprint "")
+    )
+    (path "/07a796a7-971a-46f8-be0a-5ed59c09f1bb/9fcbc6c1-ce32-4c86-9945-a29a7439aa1b"
+      (reference "#GND033") (unit 1) (value "GND") (footprint "")
+    )
+    (path "/07a796a7-971a-46f8-be0a-5ed59c09f1bb/5524fb7f-b411-428d-8611-d6ed948eb3ee"
+      (reference "#GND034") (unit 1) (value "GND") (footprint "")
+    )
     (path "/e833bd32-6ac8-4a98-bae6-223e3ec7ed32"
       (reference "#PWR01") (unit 1) (value "+3.3V") (footprint "")
@@
       (reference "C36") (unit 1) (value "4.7uF_100V") (footprint "")
     )
+    (path "/07a796a7-971a-46f8-be0a-5ed59c09f1bb/8071e84e-81fb-4f20-bf86-f86355ce3695"
+      (reference "C37") (unit 1) (value "100n") (footprint "")
+    )
+    (path "/07a796a7-971a-46f8-be0a-5ed59c09f1bb/ef7b546d-3d75-47b7-b259-64ea705e0e28"
+      (reference "C38") (unit 1) (value "100n") (footprint "")
+    )
+    (path "/07a796a7-971a-46f8-be0a-5ed59c09f1bb/fbfaa32f-35f6-4fd8-98d3-867e6001b846"
+      (reference "C39") (unit 1) (value "100n") (footprint "")
+    )
     (path "/823fda34-25a4-415d-8b6e-532f959c1c21/a8cb29ab-a205-4107-a8fa-c5105c34d4bf"
