File: Design/hall_filters.kicad_sch (KiCad schematic)
At the start: 11 parts

Commit message: SWD debugger
Parts:
- removed C? (x3): 4.7nF, symbol Device:C
- removed R? (x3): 10k, symbol Device:R
Changed lines of the file:
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@@
   (junction (at 94.615 68.58) (diameter 0) (color 0 0 0 0)
   )
-  (junction (at 140.335 68.58) (diameter 0) (color 0 0 0 0)
-  )
   (junction (at 75.565 41.91) (diameter 0) (color 0 0 0 0)
-  )
-  (junction (at 118.745 60.96) (diameter 0) (color 0 0 0 0)
-  )
-  (junction (at 129.54 64.77) (diameter 0) (color 0 0 0 0)
   )
   (junction (at 81.915 60.96) (diameter 0) (color 0 0 0 0)
@@
   (junction (at 88.265 41.91) (diameter 0) (color 0 0 0 0)
   )
-  (wire (pts (xy 118.745 84.455) (xy 118.745 89.535))
-    (stroke (width 0) (type default) (color 0 0 0 0))
-  )
   (wire (pts (xy 75.565 41.91) (xy 75.565 44.45))
     (stroke (width 0) (type default) (color 0 0 0 0))
   )
-  (wire (pts (xy 129.54 64.77) (xy 153.035 64.77))
+  (wire (pts (xy 88.265 64.77) (xy 153.035 64.77))
     (stroke (width 0) (type default) (color 0 0 0 0))
   )
@@
     (stroke (width 0) (type default) (color 0 0 0 0))
   )
-  (wire (pts (xy 81.915 60.96) (xy 105.41 60.96))
-    (stroke (width 0) (type default) (color 0 0 0 0))
-  )
-  (wire (pts (xy 129.54 84.455) (xy 129.54 89.535))
-    (stroke (width 0) (type default) (color 0 0 0 0))
-  )
   (wire (pts (xy 75.565 72.39) (xy 153.035 72.39))
-    (stroke (width 0) (type default) (color 0 0 0 0))
-  )
-  (wire (pts (xy 113.03 64.77) (xy 129.54 64.77))
-    (stroke (width 0) (type default) (color 0 0 0 0))
-  )
-  (wire (pts (xy 88.265 64.77) (xy 105.41 64.77))
-    (stroke (width 0) (type default) (color 0 0 0 0))
-  )
-  (wire (pts (xy 140.335 68.58) (xy 140.335 76.835))
-    (stroke (width 0) (type default) (color 0 0 0 0))
-  )
-  (wire (pts (xy 129.54 64.77) (xy 129.54 76.835))
     (stroke (width 0) (type default) (color 0 0 0 0))
   )
@@
     (stroke (width 0) (type default) (color 0 0 0 0))
   )
-  (wire (pts (xy 113.03 60.96) (xy 118.745 60.96))
+  (wire (pts (xy 81.915 60.96) (xy 153.035 60.96))
     (stroke (width 0) (type default) (color 0 0 0 0))
   )
-  (wire (pts (xy 140.335 68.58) (xy 153.035 68.58))
+  (wire (pts (xy 94.615 68.58) (xy 153.035 68.58))
     (stroke (width 0) (type default) (color 0 0 0 0))
   )
   (wire (pts (xy 75.565 84.455) (xy 75.565 89.535))
-    (stroke (width 0) (type default) (color 0 0 0 0))
-  )
-  (wire (pts (xy 94.615 68.58) (xy 105.41 68.58))
-    (stroke (width 0) (type default) (color 0 0 0 0))
-  )
-  (wire (pts (xy 140.335 84.455) (xy 140.335 89.535))
     (stroke (width 0) (type default) (color 0 0 0 0))
   )
@@
   )
   (wire (pts (xy 94.615 44.45) (xy 94.615 41.91))
-    (stroke (width 0) (type default) (color 0 0 0 0))
-  )
-  (wire (pts (xy 113.03 68.58) (xy 140.335 68.58))
     (stroke (width 0) (type default) (color 0 0 0 0))
   )
@@
     (stroke (width 0) (type default) (color 0 0 0 0))
   )
-  (wire (pts (xy 118.745 60.96) (xy 153.035 60.96))
-    (stroke (width 0) (type default) (color 0 0 0 0))
-  )
   (wire (pts (xy 94.615 68.58) (xy 94.615 52.07))
-    (stroke (width 0) (type default) (color 0 0 0 0))
-  )
-  (wire (pts (xy 118.745 60.96) (xy 118.745 76.835))
     (stroke (width 0) (type default) (color 0 0 0 0))
   )
@@
   (hierarchical_label "HALL1_OUT" (shape output) (at 153.035 68.58 0)
     (effects (font (size 1.27 1.27)) (justify left))
-  )
-  (symbol (lib_id "power:GND") (at 140.335 89.535 0) (unit 1)
-    (in_bom yes) (on_board yes) (fields_autoplaced)
-    (property "Reference" "#GND" (id 0) (at 140.335 95.885 0)
-      (effects (font (size 1.27 1.27)) hide)
-    )
-    (property "Value" "GND" (id 1) (at 140.335 93.98 0)
-      (effects (font (size 1.27 1.27)) hide)
-    )
-    (property "Footprint" "" (id 2) (at 140.335 89.535 0)
-      (effects (font (size 1.27 1.27)) hide)
-    )
-    (property "Datasheet" "" (id 3) (at 140.335 89.535 0)
-      (effects (font (size 1.27 1.27)) hide)
-    )
-    (pin "1")
   )
   (symbol (lib_id "Device:R") (at 88.265 48.26 0) (unit 1)
@@
     (pin "1")
   )
-  (symbol (lib_id "Device:C") (at 129.54 80.645 0) (unit 1)
-    (in_bom yes) (on_board yes)
-    (property "Reference" "C?" (id 0) (at 130.175 78.105 0)
-      (effects (font (size 1.27 1.27)) (justify left))
-    )
-    (property "Value" "4.7nF" (id 1) (at 130.175 83.185 0)
-      (effects (font (size 1.27 1.27)) (justify left))
-    )
-    (property "Footprint" "" (id 2) (at 130.5052 84.455 0)
-      (effects (font (size 1.27 1.27)) hide)
-    )
-    (property "Datasheet" "~" (id 3) (at 129.54 80.645 0)
-      (effects (font (size 1.27 1.27)) hide)
-    )
-    (pin "1")
-    (pin "2")
-  )
-  (symbol (lib_id "Device:R") (at 109.22 64.77 90) (unit 1)
-    (in_bom yes) (on_board yes)
-    (property "Reference" "R?" (id 0) (at 104.775 63.5 90))
-    (property "Value" "10k" (id 1) (at 109.22 64.77 90))
-    (property "Footprint" "" (id 2) (at 109.22 66.548 90)
-      (effects (font (size 1.27 1.27)) hide)
-    )
-    (property "Datasheet" "~" (id 3) (at 109.22 64.77 0)
-      (effects (font (size 1.27 1.27)) hide)
-    )
-    (pin "1")
-    (pin "2")
-  )
-  (symbol (lib_id "Device:R") (at 109.22 68.58 90) (unit 1)
-    (in_bom yes) (on_board yes)
-    (property "Reference" "R?" (id 0) (at 104.775 67.31 90))
-    (property "Value" "10k" (id 1) (at 109.22 68.58 90))
-    (property "Footprint" "" (id 2) (at 109.22 70.358 90)
-      (effects (font (size 1.27 1.27)) hide)
-    )
-    (property "Datasheet" "~" (id 3) (at 109.22 68.58 0)
-      (effects (font (size 1.27 1.27)) hide)
-    )
-    (pin "1")
-    (pin "2")
-  )
   (symbol (lib_id "Device:R") (at 75.565 48.26 0) (unit 1)
     (in_bom yes) (on_board yes)
@@
     (pin "1")
     (pin "2")
-  )
-  (symbol (lib_id "Device:R") (at 109.22 60.96 90) (unit 1)
-    (in_bom yes) (on_board yes)
-    (property "Reference" "R?" (id 0) (at 104.775 59.69 90))
-    (property "Value" "10k" (id 1) (at 109.22 60.96 90))
-    (property "Footprint" "" (id 2) (at 109.22 62.738 90)
-      (effects (font (size 1.27 1.27)) hide)
-    )
-    (property "Datasheet" "~" (id 3) (at 109.22 60.96 0)
-      (effects (font (size 1.27 1.27)) hide)
-    )
-    (pin "1")
-    (pin "2")
-  )
-  (symbol (lib_id "power:GND") (at 129.54 89.535 0) (unit 1)
-    (in_bom yes) (on_board yes) (fields_autoplaced)
-    (property "Reference" "#GND" (id 0) (at 129.54 95.885 0)
-      (effects (font (size 1.27 1.27)) hide)
-    )
-    (property "Value" "GND" (id 1) (at 129.54 93.98 0)
-      (effects (font (size 1.27 1.27)) hide)
-    )
-    (property "Footprint" "" (id 2) (at 129.54 89.535 0)
-      (effects (font (size 1.27 1.27)) hide)
-    )
-    (property "Datasheet" "" (id 3) (at 129.54 89.535 0)
-      (effects (font (size 1.27 1.27)) hide)
-    )
-    (pin "1")
   )
   (symbol (lib_id "Device:R") (at 81.915 48.26 0) (unit 1)
@@
     (pin "2")
   )
-  (symbol (lib_id "Device:C") (at 140.335 80.645 0) (unit 1)
-    (in_bom yes) (on_board yes)
-    (property "Reference" "C?" (id 0) (at 140.97 78.105 0)
-      (effects (font (size 1.27 1.27)) (justify left))
-    )
-    (property "Value" "4.7nF" (id 1) (at 140.97 83.185 0)
-      (effects (font (size 1.27 1.27)) (justify left))
-    )
-    (property "Footprint" "" (id 2) (at 141.3002 84.455 0)
-      (effects (font (size 1.27 1.27)) hide)
-    )
-    (property "Datasheet" "~" (id 3) (at 140.335 80.645 0)
-      (effects (font (size 1.27 1.27)) hide)
-    )
-    (pin "1")
-    (pin "2")
-  )
-  (symbol (lib_id "power:GND") (at 118.745 89.535 0) (unit 1)
-    (in_bom yes) (on_board yes) (fields_autoplaced)
-    (property "Reference" "#GND" (id 0) (at 118.745 95.885 0)
-      (effects (font (size 1.27 1.27)) hide)
-    )
-    (property "Value" "GND" (id 1) (at 118.745 93.98 0)
-      (effects (font (size 1.27 1.27)) hide)
-    )
-    (property "Footprint" "" (id 2) (at 118.745 89.535 0)
-      (effects (font (size 1.27 1.27)) hide)
-    )
-    (property "Datasheet" "" (id 3) (at 118.745 89.535 0)
-      (effects (font (size 1.27 1.27)) hide)
-    )
-    (pin "1")
-  )
   (symbol (lib_id "Device:C") (at 75.565 80.645 0) (unit 1)
     (in_bom yes) (on_board yes)
@@
       (effects (font (size 1.27 1.27)) hide)
     )
-    (pin "1")
-    (pin "2")
-  )
-  (symbol (lib_id "Device:C") (at 118.745 80.645 0) (unit 1)
-    (in_bom yes) (on_board yes)
-    (property "Reference" "C?" (id 0) (at 119.38 78.105 0)
-      (effects (font (size 1.27 1.27)) (justify left))
-    )
-    (property "Value" "4.7nF" (id 1) (at 119.38 83.185 0)
-      (effects (font (size 1.27 1.27)) (justify left))
-    )
-    (property "Footprint" "" (id 2) (at 119.7102 84.455 0)
-      (effects (font (size 1.27 1.27)) hide)
-    )
-    (property "Datasheet" "~" (id 3) (at 118.745 80.645 0)
-      (effects (font (size 1.27 1.27)) hide)
-    )

Commit message: Updating schematic
Parts:
- C3: renamed from C?; value 100nF -> 100n
- gave numbers to parts that had none: 4
Changed lines of the file:
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@@
   (symbol (lib_id "Device:R") (at 88.265 48.26 0) (unit 1)
     (in_bom yes) (on_board yes)
-    (property "Reference" "R?" (id 0) (at 86.36 49.53 90)
+    (property "Reference" "R6" (id 0) (at 86.36 49.53 90)
       (effects (font (size 1.27 1.27)) (justify left))
     )
@@
   (symbol (lib_id "Device:R") (at 94.615 48.26 0) (unit 1)
     (in_bom yes) (on_board yes)
-    (property "Reference" "R?" (id 0) (at 92.71 49.53 90)
+    (property "Reference" "R7" (id 0) (at 92.71 49.53 90)
       (effects (font (size 1.27 1.27)) (justify left))
     )
@@
   (symbol (lib_id "power:+3.3V") (at 75.565 38.735 0) (unit 1)
     (in_bom yes) (on_board yes)
-    (property "Reference" "#PWR3.3" (id 0) (at 75.565 42.545 0)
+    (property "Reference" "#PWR06" (id 0) (at 75.565 42.545 0)
       (effects (font (size 1.27 1.27)) hide)
     )
@@
   (symbol (lib_id "Device:R") (at 75.565 48.26 0) (unit 1)
     (in_bom yes) (on_board yes)
-    (property "Reference" "R?" (id 0) (at 73.66 49.53 90)
+    (property "Reference" "R4" (id 0) (at 73.66 49.53 90)
       (effects (font (size 1.27 1.27)) (justify left))
     )
@@
   (symbol (lib_id "Device:R") (at 81.915 48.26 0) (unit 1)
     (in_bom yes) (on_board yes)
-    (property "Reference" "R?" (id 0) (at 80.01 49.53 90)
+    (property "Reference" "R5" (id 0) (at 80.01 49.53 90)
       (effects (font (size 1.27 1.27)) (justify left))
     )
@@
   (symbol (lib_id "Device:C") (at 75.565 80.645 0) (unit 1)
     (in_bom yes) (on_board yes)
-    (property "Reference" "C?" (id 0) (at 76.2 78.105 0)
+    (property "Reference" "C3" (id 0) (at 76.2 78.105 0)
       (effects (font (size 1.27 1.27)) (justify left))
     )
-    (property "Value" "100nF" (id 1) (at 76.2 83.185 0)
+    (property "Value" "100n" (id 1) (at 76.2 83.185 0)
       (effects (font (size 1.27 1.27)) (justify left))
     )
@@
   (symbol (lib_id "power:GND") (at 75.565 89.535 0) (unit 1)
     (in_bom yes) (on_board yes) (fields_autoplaced)
-    (property "Reference" "#GND" (id 0) (at 75.565 95.885 0)
+    (property "Reference" "#GND09" (id 0) (at 75.565 95.885 0)
       (effects (font (size 1.27 1.27)) hide)
     )

Commit message: adding caps
Parts:
- added C37, C38, C39: 100n, symbol Device:C
Connections:
- net GND: now also C37.2, C38.2, C39.2
- net HALL1_IN: now also C39.1
- net HALL2_IN: now also C38.1
- net HALL3_IN: now also C37.1
Changed lines of the file:
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@@
   (junction (at 88.265 64.77) (diameter 0) (color 0 0 0 0)
   )
+  (junction (at 108.585 60.96) (diameter 0) (color 0 0 0 0)
+  )
+  (junction (at 126.365 68.58) (diameter 0) (color 0 0 0 0)
+  )
   (junction (at 94.615 68.58) (diameter 0) (color 0 0 0 0)
   )
@@
   (junction (at 81.915 60.96) (diameter 0) (color 0 0 0 0)
   )
+  (junction (at 117.475 64.77) (diameter 0) (color 0 0 0 0)
+  )
   (junction (at 88.265 41.91) (diameter 0) (color 0 0 0 0)
   )
@@
     (stroke (width 0) (type default) (color 0 0 0 0))
   )
-  (wire (pts (xy 88.265 64.77) (xy 153.035 64.77))
+  (wire (pts (xy 88.265 64.77) (xy 117.475 64.77))
+    (stroke (width 0) (type default) (color 0 0 0 0))
+  )
+  (wire (pts (xy 126.365 68.58) (xy 126.365 76.835))
     (stroke (width 0) (type default) (color 0 0 0 0))
   )
@@
     (stroke (width 0) (type default) (color 0 0 0 0))
   )
+  (wire (pts (xy 117.475 64.77) (xy 117.475 76.835))
+    (stroke (width 0) (type default) (color 0 0 0 0))
+  )
   (wire (pts (xy 75.565 72.39) (xy 153.035 72.39))
     (stroke (width 0) (type default) (color 0 0 0 0))
   )
+  (wire (pts (xy 108.585 60.96) (xy 108.585 76.835))
+    (stroke (width 0) (type default) (color 0 0 0 0))
+  )
+  (wire (pts (xy 126.365 68.58) (xy 153.035 68.58))
+    (stroke (width 0) (type default) (color 0 0 0 0))
+  )
+  (wire (pts (xy 117.475 64.77) (xy 153.035 64.77))
+    (stroke (width 0) (type default) (color 0 0 0 0))
+  )
   (wire (pts (xy 81.915 41.91) (xy 75.565 41.91))
     (stroke (width 0) (type default) (color 0 0 0 0))
@@
     (stroke (width 0) (type default) (color 0 0 0 0))
   )
-  (wire (pts (xy 81.915 60.96) (xy 153.035 60.96))
-    (stroke (width 0) (type default) (color 0 0 0 0))
-  )
-  (wire (pts (xy 94.615 68.58) (xy 153.035 68.58))
+  (wire (pts (xy 81.915 60.96) (xy 108.585 60.96))
+    (stroke (width 0) (type default) (color 0 0 0 0))
+  )
+  (wire (pts (xy 94.615 68.58) (xy 126.365 68.58))
     (stroke (width 0) (type default) (color 0 0 0 0))
   )
@@
     (stroke (width 0) (type default) (color 0 0 0 0))
   )
+  (wire (pts (xy 126.365 84.455) (xy 126.365 89.535))
+    (stroke (width 0) (type default) (color 0 0 0 0))
+  )
   (wire (pts (xy 88.265 64.77) (xy 88.265 52.07))
     (stroke (width 0) (type default) (color 0 0 0 0))
@@
     (stroke (width 0) (type default) (color 0 0 0 0))
   )
+  (wire (pts (xy 117.475 84.455) (xy 117.475 89.535))
+    (stroke (width 0) (type default) (color 0 0 0 0))
+  )
   (wire (pts (xy 57.15 68.58) (xy 94.615 68.58))
     (stroke (width 0) (type default) (color 0 0 0 0))
   )
   (wire (pts (xy 88.265 41.91) (xy 81.915 41.91))
+    (stroke (width 0) (type default) (color 0 0 0 0))
+  )
+  (wire (pts (xy 108.585 84.455) (xy 108.585 89.535))
+    (stroke (width 0) (type default) (color 0 0 0 0))
+  )
+  (wire (pts (xy 108.585 60.96) (xy 153.035 60.96))
     (stroke (width 0) (type default) (color 0 0 0 0))
   )
@@
     (pin "2")
   )
+  (symbol (lib_id "power:GND") (at 126.365 89.535 0) (unit 1)
+    (in_bom yes) (on_board yes) (fields_autoplaced)
+    (property "Reference" "#GND034" (id 0) (at 126.365 95.885 0)
+      (effects (font (size 1.27 1.27)) hide)
+    )
+    (property "Value" "GND" (id 1) (at 126.365 93.98 0)
+      (effects (font (size 1.27 1.27)) hide)
+    )
+    (property "Footprint" "" (id 2) (at 126.365 89.535 0)
+      (effects (font (size 1.27 1.27)) hide)
+    )
+    (property "Datasheet" "" (id 3) (at 126.365 89.535 0)
+      (effects (font (size 1.27 1.27)) hide)
+    )
+    (pin "1")
+  )
+  (symbol (lib_id "power:GND") (at 108.585 89.535 0) (unit 1)
+    (in_bom yes) (on_board yes) (fields_autoplaced)
+    (property "Reference" "#GND032" (id 0) (at 108.585 95.885 0)
+      (effects (font (size 1.27 1.27)) hide)
+    )
+    (property "Value" "GND" (id 1) (at 108.585 93.98 0)
+      (effects (font (size 1.27 1.27)) hide)
+    )
+    (property "Footprint" "" (id 2) (at 108.585 89.535 0)
+      (effects (font (size 1.27 1.27)) hide)
+    )
+    (property "Datasheet" "" (id 3) (at 108.585 89.535 0)
+      (effects (font (size 1.27 1.27)) hide)
+    )
+    (pin "1")
+  )
+  (symbol (lib_id "Device:C") (at 108.585 80.645 0) (unit 1)
+    (in_bom yes) (on_board yes)
+    (property "Reference" "C37" (id 0) (at 109.22 78.105 0)
+      (effects (font (size 1.27 1.27)) (justify left))
+    )
+    (property "Value" "100n" (id 1) (at 109.22 83.185 0)
+      (effects (font (size 1.27 1.27)) (justify left))
+    )
+    (property "Footprint" "" (id 2) (at 109.5502 84.455 0)
+      (effects (font (size 1.27 1.27)) hide)
+    )
+    (property "Datasheet" "~" (id 3) (at 108.585 80.645 0)
+      (effects (font (size 1.27 1.27)) hide)
+    )
+    (pin "1")
+    (pin "2")
+  )
   (symbol (lib_id "Device:R") (at 81.915 48.26 0) (unit 1)
     (in_bom yes) (on_board yes)
@@
     (pin "1")
     (pin "2")
+  )
+  (symbol (lib_id "power:GND") (at 117.475 89.535 0) (unit 1)
+    (in_bom yes) (on_board yes) (fields_autoplaced)
+    (property "Reference" "#GND033" (id 0) (at 117.475 95.885 0)
+      (effects (font (size 1.27 1.27)) hide)
+    )
+    (property "Value" "GND" (id 1) (at 117.475 93.98 0)
+      (effects (font (size 1.27 1.27)) hide)
+    )
+    (property "Footprint" "" (id 2) (at 117.475 89.535 0)
+      (effects (font (size 1.27 1.27)) hide)
+    )
+    (property "Datasheet" "" (id 3) (at 117.475 89.535 0)
+      (effects (font (size 1.27 1.27)) hide)
+    )
+    (pin "1")
   )
   (symbol (lib_id "Device:C") (at 75.565 80.645 0) (unit 1)
@@
     (pin "1")
   )
+  (symbol (lib_id "Device:C") (at 117.475 80.645 0) (unit 1)
+    (in_bom yes) (on_board yes)
+    (property "Reference" "C38" (id 0) (at 118.11 78.105 0)
+      (effects (font (size 1.27 1.27)) (justify left))
+    )
+    (property "Value" "100n" (id 1) (at 118.11 83.185 0)
+      (effects (font (size 1.27 1.27)) (justify left))
+    )
+    (property "Footprint" "" (id 2) (at 118.4402 84.455 0)
+      (effects (font (size 1.27 1.27)) hide)
+    )
+    (property "Datasheet" "~" (id 3) (at 117.475 80.645 0)
+      (effects (font (size 1.27 1.27)) hide)
+    )
+    (pin "1")
+    (pin "2")
+  )
+  (symbol (lib_id "Device:C") (at 126.365 80.645 0) (unit 1)
+    (in_bom yes) (on_board yes)
+    (property "Reference" "C39" (id 0) (at 127 78.105 0)
+      (effects (font (size 1.27 1.27)) (justify left))
+    )
+    (property "Value" "100n" (id 1) (at 127 83.185 0)
+      (effects (font (size 1.27 1.27)) (justify left))
+    )
+    (property "Footprint" "" (id 2) (at 127.3302 84.455 0)
+      (effects (font (size 1.27 1.27)) hide)
+    )
+    (property "Datasheet" "~" (id 3) (at 126.365 80.645 0)
+      (effects (font (size 1.27 1.27)) hide)
+    )
+    (pin "1")
+    (pin "2")
+  )
 )
